Commit message: Add files via upload

File: src/my_robot_description/urdf/my_robot.urdf.xacro (robot description, xacro)
@@ -4,3 +4,5 @@
      <xacro:include filename="robot_base.xacro"/>
      <xacro:include filename="robot_base_gazebo.xacro"/>
+     <xacro:include filename="camera.xacro"/>
+     <xacro:include filename="lidar.xacro"/>
 </robot>

File: src/my_robot_description/urdf/robot_base.xacro (robot description, xacro)
@@ -2,10 +2,10 @@
 <robot xmlns:xacro ="http://www.ros.org/wiki/xacro">
      <!-- Robot Properties -->
-    <xacro:property name="base_length" value="5"/>  lenght of base divided by 10
-    <xacro:property name="base_width" value="3.5"/> width of base divided by 10
-    <xacro:property name="base_height" value="1"/>  height of base  divided by 10
-    <xacro:property name="radius_wheels" value="0.8"/>
-    <xacro:property name="thick_wheels" value="0.3"/>
-    <xacro:property name="wheel_joint_hieght" value="0.3"/>
+    <xacro:property name="base_length" value="0.5"/>  lenght of base divided by 10
+    <xacro:property name="base_width" value="0.35"/> width of base divided by 10
+    <xacro:property name="base_height" value="0.1"/>  height of base  divided by 10
+    <xacro:property name="radius_wheels" value="0.08"/>
+    <xacro:property name="thick_wheels" value="0.03"/>
+    <xacro:property name="wheel_joint_hieght" value="0.03"/>
     <!-- Base Footprint -->
     <link name="base_footprint"/>
@@ -58,5 +58,5 @@
         <parent link="base_footprint"/>
         <child link="base_link"/>
-        <origin xyz="0 0 0.5" rpy="0 0 0"/>  0.5 diffrent  between
+        <origin xyz="0 0 0.05" rpy="0 0 0"/>  0.05 diffrent  between
     </joint>
     <!-- Continuous Joints for Wheels -->
@@ -65,5 +65,5 @@
         <parent link="base_link"/>
         <child link ="right_r_wheel_link"/>
-        <origin xyz="-1.8 -1.9 ${wheel_joint_hieght}" rpy="0 0 0"/> ///distance between center and wheel
+        <origin xyz="-0.18 -0.19 ${wheel_joint_hieght}" rpy="0 0 0"/> ///distance between center and wheel
         <axis xyz="0 1 0"/>
     </joint>
@@ -72,5 +72,5 @@
         <parent link="base_link"/>
         <child link="right_f_wheel_link"/>
-        <origin xyz="1.8 -1.9 ${wheel_joint_hieght}" rpy="0 0 0"/>
+        <origin xyz="0.18 -0.19 ${wheel_joint_hieght}" rpy="0 0 0"/>
         <axis xyz="0 1 0"/>
     </joint>
@@ -79,5 +79,5 @@
         <parent link="base_link"/>
         <child link="left_r_wheel_link"/>
-        <origin xyz="-1.8 1.9 ${wheel_joint_hieght}" rpy="0 0 0"/>
+        <origin xyz="-0.18 0.19 ${wheel_joint_hieght}" rpy="0 0 0"/>
         <axis xyz="0 1 0"/>
     </joint>
@@ -86,5 +86,5 @@
         <parent link="base_link"/>
         <child link="left_f_wheel_link"/>
-        <origin xyz="1.8 1.9 ${wheel_joint_hieght}" rpy="0 0 0"/>
+        <origin xyz="0.18 0.19 ${wheel_joint_hieght}" rpy="0 0 0"/>
         <axis xyz="0 1 0"/>
     </joint>
